File: meishi_tenkey.kicad_pcb (KiCad board)
At the start: 2 copper layers, 55 x 91 mm, 45 parts, among them J1 Conn_01x07_Socket, J2 Conn_01x07_Socket, J3 Conn_01x07_Pin, J4 Conn_01x07_Pin, SW1 SW_Push, SW10 SW_Push, SW11 SW_Push, SW12 SW_Push, SW13 SW_Push, SW14 SW_Push, SW15 SW_Push, SW16 SW_Push, SW17 SW_Push, SW18 SW_Push, SW19 SW_Push, SW2 SW_Push, SW20 SW_Push, SW3 SW_Push, SW4 SW_Push, SW5 SW_Push, SW6 SW_Push, SW7 SW_Push, SW8 SW_Push, SW9 SW_Push, U1 XIAO-RP2040-SMD

Commit message: fix: correct MCU through-hole pitch in footprint (v0.2)
Fix incorrect through-hole spacing for the microcontroller footprint.
Regenerate all gerber files with the corrected PCB design.
Update README to note the fix for v0.1 users.

Co-Authored-By: Claude Opus 4.6 <noreply@anthropic.com>
Parts:
- removed J1, J2: Conn_01x07_Socket, Connector_PinSocket_2.54mm:PinSocket_1x07_P2.54mm_Vertical
- removed J3, J4: Conn_01x07_Pin, Connector_PinHeader_2.54mm:PinHeader_1x07_P2.54mm_Vertical
- U1: value XIAO-RP2040-SMD -> XIAO-RP2040-DIP; footprint Seeed Studio XIAO Series Library:XIAO-RP2040-SMD -> Seeed Studio XIAO Series Library:XIAO-RP2040-DIP
- moved U1 61.1 mm to (171.4, 48.5)
Connections:
- U1 pad 1: Net-(J3-Pin_1) -> Row0
- U1 pad 10: Net-(J4-Pin_5) -> Col1
- U1 pad 11: Net-(J4-Pin_4) -> Col0
- U1 pad 12: Net-(J4-Pin_3) -> unconnected-(U1-3V3-Pad12)
- U1 pad 13: Net-(J4-Pin_2) -> unconnected-(U1-GND-Pad13)
- U1 pad 14: Net-(J4-Pin_1) -> unconnected-(U1-VBUS-Pad14)
- U1 pad 2: Net-(J3-Pin_2) -> Row1
- U1 pad 3: Net-(J3-Pin_3) -> Row2
- U1 pad 4: Net-(J3-Pin_4) -> Row3
- U1 pad 5: Net-(J3-Pin_5) -> Row4
- U1 pad 6: Net-(J3-Pin_6) -> unconnected-(U1-GPIO7/SCL-Pad6)
- U1 pad 7: Net-(J3-Pin_7) -> unconnected-(U1-GPIO0/TX-Pad7)
- U1 pad 8: Net-(J4-Pin_7) -> Col3
- U1 pad 9: Net-(J4-Pin_6) -> Col2
Routing:
- net Net-(J3-Pin_7): track 8.56 -> 0.00 mm
- net Net-(J3-Pin_6): track 8.56 -> 0.00 mm
- net Net-(J3-Pin_5): track 8.56 -> 0.00 mm
- net Net-(J3-Pin_4): track 8.56 -> 0.00 mm
- net Net-(J3-Pin_3): track 8.56 -> 0.00 mm
- net Net-(J3-Pin_2): track 8.56 -> 0.00 mm
- net Net-(J3-Pin_1): track 8.56 -> 0.00 mm
- net Net-(J4-Pin_7): track 7.30 -> 0.00 mm
- net Net-(J4-Pin_6): track 7.30 -> 0.00 mm
- net Net-(J4-Pin_5): track 7.30 -> 0.00 mm
- net Net-(J4-Pin_4): track 7.30 -> 0.00 mm
- net Net-(J4-Pin_3): track 7.30 -> 0.00 mm
- net Net-(J4-Pin_2): track 7.30 -> 0.00 mm
- net Net-(J4-Pin_1): track 7.30 -> 0.00 mm
Other:
- board text added: "meishi_tenky ver.0.2"
- board text removed: "meishi_tenky ver.0.1"
